Commit message: add map

File: project/proj3_fly/rsc/HextechUAV.urdf (robot description, URDF)
Before this commit: robot HextechUAV, 6 links, 5 joints
Joints:
- joint World2Zaxis: limit lower=-10.0 upper=10.0 effort=0.0 velocity=100.0 -> lower=-8.0 upper=8.0 effort=0.0 velocity=100.0
- joint Zaxis2Xaxis: limit lower=-100.0 upper=100.0 effort=0.0 velocity=100.0 -> lower=-18 upper=16 effort=0.0 velocity=100.0

File: project/proj3_fly/rsc/forest.urdf (robot description, URDF)
Before this commit: robot forest, 2 links, 1 joints
Links:
- added link obstacle_0, mass 1.0; collision box size=2 2 2; visual box size=2 2 2
- added link obstacle_10, mass 1.0; collision box size=1.8213203435596428 2 1.8213203435596428; visual box size=1.8213203435596428 2 1.8213203435596428
- added link obstacle_11, mass 1.0; collision box size=1.8213203435596428 2 1.8213203435596428; visual box size=1.8213203435596428 2 1.8213203435596428
- added link obstacle_12, mass 1.0; collision box size=40 2 2; visual box size=40 2 2
- added link obstacle_13, mass 1.0; collision box size=40 2 2; visual box size=40 2 2
- added link obstacle_2, mass 1.0; collision box size=2 2 8; visual box size=2 2 8
- added link obstacle_3, mass 1.0; collision box size=2 2 6; visual box size=2 2 6
- added link obstacle_4, mass 1.0; collision box size=2 2 4; visual box size=2 2 4
- added link obstacle_5, mass 1.0; collision box size=2 2 6; visual box size=2 2 6
- added link obstacle_6, mass 1.0; collision box size=2 2 12; visual box size=2 2 12
- added link obstacle_7, mass 1.0; collision box size=2 2 2; visual box size=2 2 2
- added link obstacle_8, mass 1.0; collision box size=2 2 4; visual box size=2 2 4
- added link obstacle_9, mass 1.0; collision box size=2 2 9.5; visual box size=2 2 9.5
- link obstacle_1: mass 10.0 -> 1.0; geometry collision box size=2 2 10; visual box size=2 2 10
Joints:
- removed joint obstacle_1_to_base
- added joint base_to_obstacle_0: type fixed, parent base, child obstacle_0, origin xyz=-11 0.9 -7 rpy=0 0 0
- added joint base_to_obstacle_1: type fixed, parent base, child obstacle_1, origin xyz=-11 0.9 3 rpy=0 0 0
- added joint base_to_obstacle_10: type fixed, parent base, child obstacle_10, origin xyz=-1 0.9 2.7121320343559643 rpy=0 0.785 0
- added joint base_to_obstacle_11: type fixed, parent base, child obstacle_11, origin xyz=1 0.9 1.2878679656440357 rpy=0 0.785 0
- added joint base_to_obstacle_12: type fixed, parent base, child obstacle_12, origin xyz=0 0.9 -9 rpy=0 0 0
- added joint base_to_obstacle_13: type fixed, parent base, child obstacle_13, origin xyz=0 0.9 9 rpy=0 0 0
- added joint base_to_obstacle_2: type fixed, parent base, child obstacle_2, origin xyz=-5 0.9 -4 rpy=0 0 0
- added joint base_to_obstacle_3: type fixed, parent base, child obstacle_3, origin xyz=-5 0.9 5 rpy=0 0 0
- added joint base_to_obstacle_4: type fixed, parent base, child obstacle_4, origin xyz=-1 0.9 6 rpy=0 0 0
- added joint base_to_obstacle_5: type fixed, parent base, child obstacle_5, origin xyz=1 0.9 -3 rpy=0 0 0
- added joint base_to_obstacle_6: type fixed, parent base, child obstacle_6, origin xyz=7 0.9 -2 rpy=0 0 0
- added joint base_to_obstacle_7: type fixed, parent base, child obstacle_7, origin xyz=7 0.9 7 rpy=0 0 0
- added joint base_to_obstacle_8: type fixed, parent base, child obstacle_8, origin xyz=11 0.9 6 rpy=0 0 0
- added joint base_to_obstacle_9: type fixed, parent base, child obstacle_9, origin xyz=11 0.9 -1.25 rpy=0 0 0
