Commit message: update map, init pos and destination

File: project/proj4_run/rsc/map.urdf (robot description, URDF)
Before this commit: robot map, 1 links, 0 joints
Links:
- link base: geometry collision mesh filename=mesh/map_concave.obj scale=1; visual mesh filename=mesh/map_concave.obj scale=1

File: project/proj4_run/rsc/target.urdf (robot description, URDF)
Before this commit: robot target, 1 links, 0 joints
Links:
- link base: geometry collision sphere radius=0.5; visual sphere radius=0.5
