Commit message: add test script for project 4

File: project/proj4_run/rsc/MarioTheRobot.urdf (robot description, URDF)
Before this commit: robot Mario, 7 links, 5 joints
Links:
- link body: mass 0.0 -> 5.0
Joints:
- added joint ZAxis2body: type continuous, parent ZAxis, child body, origin xyz=0.0 0.0 0.0 rpy=0.0 0.0 0.0, axis 0.0 1.0 0.0
- joint World2XAxis: child Xaxis -> XAxis
- joint XAxis2ZAxis: axis 0.0 0.0 1.0 -> 0.0 0.0 -1.0; limit lower=-10.0 upper=20.0 -> lower=-10.0 upper=10.0
- joint body2thigh: axis 0.0 1.0 0.0 -> (none); type continuous -> fixed
- joint engine2: limit lower=0.0 upper=0.0 effort=0.0 velocity=0.0 -> (none)

File: project/proj4_run/rsc/target.urdf (robot description, URDF)
Before this commit: robot map, 1 links, 0 joints
Links:
- link base: geometry collision sphere radius=0.1; visual sphere radius=1.0

Commit message: Add map

File: project/proj4_run/rsc/MarioTheRobot.urdf (robot description, URDF)
Before this commit: robot Mario, 7 links, 6 joints
Links:
- link wheel: mass 0.5 -> 1.0

File: project/proj4_run/rsc/map.urdf (robot description, URDF)
Before this commit: robot map, 1 links, 0 joints
Links:
- link base: geometry collision mesh filename=mesh/map.STL scale=1.0; visual mesh filename=mesh/map.STL scale=1.0

Commit message: use v-hacd to make a concave map

File: project/proj4_run/rsc/MarioTheRobot.urdf (robot description, URDF)
Before this commit: robot Mario, 7 links, 6 joints
Links:
- link body: geometry collision box size=0.3 0.2 0.2; visual box size=0.3 0.2 0.2
Joints:
- joint XAxis2ZAxis: limit lower=-10.0 upper=10.0 -> lower=-50.0 upper=50.0

Commit message: add velocity limitation to engines

File: project/proj4_run/rsc/MarioTheRobot.urdf (robot description, URDF)
Before this commit: robot Mario, 7 links, 6 joints
Joints:
- joint engine1: limit (none) -> velocity=30.0
- joint engine2: limit (none) -> velocity=30.0
